Commit message: fixed the controller. Needed to add continous joints at the front

File: src/robot_description/urdf/robot_core.xacro (robot description, xacro)
@@ -31,5 +31,5 @@
     </xacro:inertial_box>
   </link>
-  <!-- Rear Left Wheel link and joint  -->
+  <!-- Rear Left Wheel link -->
   <link name="rear_left_wheel_link">
     <visual>
@@ -50,11 +50,5 @@
     </xacro:inertial_cylinder>
   </link>
-  <joint name="rear_left_wheel_joint" type="continuous">
-    <parent link="base_link" />
-    <child link="rear_left_wheel_link" />
-    <origin xyz="-${box_length/2} ${(box_width/2)+(wheel_length/2)} -${box_height/2}" rpy="-${3.14159/2} 0 0" />
-    <axis xyz="0 0 1" />
-  </joint>
-  <!-- Rear right wheel link and joint -->
+  <!-- Rear right wheel link -->
   <link name="rear_right_wheel_link">
     <visual>
@@ -75,11 +69,5 @@
     </xacro:inertial_cylinder>
   </link>
-  <joint name="rear_right_wheel_joint" type="continuous">
-    <parent link="base_link" />
-    <child link="rear_right_wheel_link" />
-    <origin xyz="-${box_length/2} -${(box_width/2)+(wheel_length/2)} -${box_height/2}" rpy="-${3.14159/2} 0 0" />
-    <axis xyz="0 0 1" />
-  </joint>
-  <!-- Front left wheel link and joint-->
+  <!-- Front left wheel link -->
   <link name="front_left_wheel_link">
     <visual>
@@ -100,12 +88,25 @@
     </xacro:inertial_cylinder>
   </link>
-  <joint name="front_left_steering_joint" type="revolute">
-    <parent link="base_link" />
-    <child link="front_left_wheel_link" />
-    <origin xyz="${box_length/2} ${(box_width/2)+(wheel_length/2)} -${box_height/2}" rpy="-${3.14159/2} 0 0" />
-    <axis xyz="0 1 0" />
-    <limit lower="-1.0" upper="1.0" effort="100" velocity="100" />
-  </joint>
-  <!-- Front right wheel link and joint-->
+  <!-- Front left wheel steering link-->
+  <link name="front_left_steering_link">
+    <visual>
+      <origin xyz="0 0 0" rpy="0 0 0" />
+      <geometry>
+        <cylinder radius="0.001" length="0.01" />
+      </geometry>
+    </visual>
+    <collision>
+      <origin xyz="0 0 0" rpy="0 0 0" />
+      <geometry>
+        <cylinder radius="0.001" length="0.01" />
+      </geometry>
+    </collision>
+    <inertial>
+      <mass value="0.01" />
+      <origin xyz="0 0 0" />
+      <inertia ixx="0.0" ixy="0.0" ixz="0.0" iyy="1.0" iyz="0.0" izz="1.0" />
+    </inertial>
+  </link>
+  <!-- Front right wheel link-->
   <link name="front_right_wheel_link">
     <visual>
@@ -126,10 +127,64 @@
     </xacro:inertial_cylinder>
   </link>
+  <!-- Front right wheel steering link-->
+  <link name="front_right_steering_link">
+    <visual>
+      <origin xyz="0 0 0" rpy="0 0 0" />
+      <geometry>
+        <cylinder radius="0.001" length="0.01" />
+      </geometry>
+    </visual>
+    <collision>
+      <origin xyz="0 0 0" rpy="0 0 0" />
+      <geometry>
+        <cylinder radius="0.001" length="0.01" />
+      </geometry>
+    </collision>
+    <inertial>
+      <mass value="0.01" />
+      <origin xyz="0 0 0" />
+      <inertia ixx="0.0" ixy="0.0" ixz="0.0" iyy="1.0" iyz="0.0" izz="1.0" />
+    </inertial>
+  </link>
+  <!-- Joints-->
+  <joint name="rear_left_wheel_joint" type="continuous">
+    <parent link="base_link" />
+    <child link="rear_left_wheel_link" />
+    <origin xyz="-${box_length/2} ${(box_width/2)+(wheel_length/2)} -${box_height/2}" rpy="-${3.14159/2} 0 0" />
+    <axis xyz="0 0 1" />
+  </joint>
+  <joint name="rear_right_wheel_joint" type="continuous">
+    <parent link="base_link" />
+    <child link="rear_right_wheel_link" />
+    <origin xyz="-${box_length/2} -${(box_width/2)+(wheel_length/2)} -${box_height/2}" rpy="-${3.14159/2} 0 0" />
+    <axis xyz="0 0 1" />
+  </joint>
+  <joint name="front_left_steering_joint" type="revolute">
+    <parent link="base_link" />
+    <child link="front_left_steering_link" />
+    <origin xyz="${box_length/2} ${(box_width/2)+(wheel_length/2)} -${box_height/2}" rpy="-${3.14159/2} 0 0" />
+    <axis xyz="0 1 0" />
+    <limit lower="-1.0" upper="1.0" effort="100" velocity="100" />
+  </joint>
+  <joint name="front_left_wheel_joint" type="continuous">
+    <parent link="front_left_steering_link" />
+    <child link="front_left_wheel_link" />
+    <origin xyz="0 0 0" rpy="0 0 0" />
+    <axis xyz="0 0 1" />
+    <limit lower="-1.0" upper="1.0" effort="100" velocity="100" />
+  </joint>
   <joint name="front_right_steering_joint" type="revolute">
     <parent link="base_link" />
-    <child link="front_right_wheel_link" />
+    <child link="front_right_steering_link" />
     <origin xyz="${box_length/2} -${(box_width/2)+(wheel_length/2)} -${(box_height/2)}" rpy="-${3.14159/2} 0 0" />
     <axis xyz="0 1 0" />
     <limit lower="-1.0" upper="1.0" effort="100" velocity="100" />
   </joint>
+  <joint name="front_right_wheel_joint" type="continuous">
+    <parent link="front_right_steering_link" />
+    <child link="front_right_wheel_link" />
+    <origin xyz="0 0 0" rpy="0 0 0" />
+    <axis xyz="0 0 1" />
+    <limit lower="-1.0" upper="1.0" effort="100" velocity="100" />
+  </joint>
 </robot>
