Commit message: mess

File: src/robot_description/urdf/materials.xacro (robot description, xacro)
@@ -16,3 +16,6 @@
     <color rgba=" 0 0 1 1" />
   </material>
+  <material name="grey">
+    <color rgba="0 0 0 0.5" />
+  </material>
 </robot>

File: src/robot_description/urdf/robot_core.xacro (robot description, xacro)
@@ -69,5 +69,5 @@
     </xacro:inertial_cylinder>
   </link>
-  <!-- Front left wheel link -->
+  <!-- Front left wheel -->
   <link name="front_left_wheel_link">
     <visual>
@@ -88,5 +88,5 @@
     </xacro:inertial_cylinder>
   </link>
-  <!-- Front left wheel steering link-->
+  <!-- Front left wheel steering -->
   <link name="front_left_steering_link">
     <visual>
@@ -105,8 +105,8 @@
       <mass value="0.01" />
       <origin xyz="0 0 0" />
-      <inertia ixx="0.0" ixy="0.0" ixz="0.0" iyy="1.0" iyz="0.0" izz="1.0" />
+      <inertia ixx="0.0" ixy="0.0" ixz="0.0" iyy="0.0" iyz="0.0" izz="0.0" />
     </inertial>
   </link>
-  <!-- Front right wheel link-->
+  <!-- Front right wheel -->
   <link name="front_right_wheel_link">
     <visual>
@@ -127,5 +127,5 @@
     </xacro:inertial_cylinder>
   </link>
-  <!-- Front right wheel steering link-->
+  <!-- Front right wheel steering -->
   <link name="front_right_steering_link">
     <visual>
@@ -144,5 +144,5 @@
       <mass value="0.01" />
       <origin xyz="0 0 0" />
-      <inertia ixx="0.0" ixy="0.0" ixz="0.0" iyy="1.0" iyz="0.0" izz="1.0" />
+      <inertia ixx="0.0" ixy="0.0" ixz="0.0" iyy="0.0" iyz="0.0" izz="0.0" />
     </inertial>
   </link>
