Commit message: Controller setup successfull. However, robot moves slowly and cant turn around.

File: src/robot_description/urdf/gazebo_parameters.xacro (robot description, xacro)
@@ -3,8 +3,8 @@
   xmlns:xacro="http://ros.org/wiki/xacro">
   <gazebo reference = "rear_right_wheel_link">
-    <mu1>100000000</mu1>
-    <mu2>1000000000</mu2>
-    <kp>1000000000000</kp>
-    <kd>1000000000000</kd>
+    <mu1>1000</mu1>
+    <mu2>1000</mu2>
+    <kp>1000</kp>
+    <kd>0.1</kd>
     <minDepth>0.001</minDepth>
     <maxVel>0.1</maxVel>
@@ -12,8 +12,8 @@
   </gazebo>
   <gazebo reference = "rear_left_wheel_link">
-    <mu1>100000000</mu1>
-    <mu2>1000000000</mu2>
-    <kp>1000000000000</kp>
-    <kd>1000000000000</kd>
+    <mu1>1000</mu1>
+    <mu2>1000</mu2>
+    <kp>1000</kp>
+    <kd>0.1</kd>
     <minDepth>0.001</minDepth>
     <maxVel>0.1</maxVel>
@@ -21,23 +21,25 @@
   </gazebo>
   <gazebo reference = "front_right_wheel_link">
-    <mu1>100000000</mu1>
-    <mu2>1000000000</mu2>
-    <kp>1000000000000</kp>
-    <kd>1000000000000</kd>
+    <mu1>1000</mu1>
+    <mu2>1000</mu2>
+    <kp>1000</kp>
+    <kd>0.1</kd>
     <minDepth>0.001</minDepth>
-    <maxVel>0.1</maxVel>
+    <maxVel>10</maxVel>
     <fdir1>1 0 0</fdir1>
   </gazebo>
   <gazebo reference = "front_left_wheel_link">
-    <mu1>100000000</mu1>
-    <mu2>1000000000</mu2>
-    <kp>1000000000000</kp>
-    <kd>1000000000000</kd>
+    <mu1>1000</mu1>
+    <mu2>1000</mu2>
+    <kp>1000</kp>
+    <kd>0.1</kd>
     <minDepth>0.001</minDepth>
-    <maxVel>0.1</maxVel>
+    <maxVel>10</maxVel>
     <fdir1>1 0 0</fdir1>
   </gazebo>
   <gazebo>
-    <plugin name="gz_ros2_control" filename="libgz_ros2_control.so"/>
+    <plugin filename ="gz_ros2_control-system" name = "gz_ros2_control::GazeboSimROS2ControlPlugin">
+      <parameters>$(find robot_controller)/config/controllers.yaml</parameters>
+    </plugin>
   </gazebo>
 </robot>

File: src/robot_description/urdf/robot_physical_properties.xacro (robot description, xacro)
@@ -7,4 +7,4 @@
   <xacro:property name="box_width" value="0.3" />
   <xacro:property name="box_height" value="0.1" />
-  <xacro:property name="box_mass" value="5.0" />
+  <xacro:property name="box_mass" value="1.0" />
 </robot>

File: src/robot_description/urdf/ros2_control.xacro (robot description, xacro)
@@ -3,5 +3,5 @@
   <ros2_control name = "RobotSystem" type = "system">
     <hardware>
-      <plugin>gz_ros2_control/GazeboSystem</plugin>
+      <plugin>gz_ros2_control/GazeboSimSystem</plugin>
     </hardware>
     <joint name="rear_left_wheel_joint">

Commit message: changed the robot model completely

File: src/robot_description/urdf/gazebo_parameters.xacro (robot description, xacro)
@@ -5,20 +5,47 @@
     <mu1>10000000</mu1>
     <mu2>10000000</mu2>
-    <kp>10000000</kp>
+    <!-- <kp>10000000</kp>
     <kd>10000000</kd>
     <minDepth>0.001</minDepth>
-    <maxVel>0.1</maxVel>
-    <fdir1>1 0 0</fdir1>
+    <maxVel>10</maxVel>
+    <fdir1>1 0 0</fdir1> -->
   </gazebo>
   <gazebo reference = "rear_left_wheel_link">
     <mu1>10000000</mu1>
     <mu2>10000000</mu2>
+    <!-- <kp>10000000</kp>
+    <kd>10000000</kd>
+    <minDepth>0.001</minDepth>
+    <maxVel>10</maxVel>
+    <fdir1>1 0 0</fdir1> -->
+  </gazebo>
+  <gazebo reference = "front_right_wheel_link">
+    <mu1>10000000</mu1>
+    <mu2>10000000</mu2>
+    <!-- <kp>10000000</kp>
+    <kd>10000000</kd>
+    <minDepth>0.001</minDepth>
+    <maxVel>10</maxVel>
+    <fdir1>1 0 0</fdir1> -->
+  </gazebo>
+  <gazebo reference = "front_left_wheel_link">
+    <mu1>10000000</mu1>
+    <mu2>10000000</mu2>
+    <!-- <kp>10000000</kp>
+    <kd>10000000</kd>
+    <minDepth>0.001</minDepth>
+    <maxVel>10</maxVel>
+    <fdir1>1 0 0</fdir1> -->
+  </gazebo>
+  <!-- <gazebo reference = "front_left_steering_link">
+    <mu1>100000000</mu1>
+    <mu2>100000000</mu2>
     <kp>10000000</kp>
     <kd>10000000</kd>
     <minDepth>0.001</minDepth>
-    <maxVel>0.1</maxVel>
+    <maxVel>10</maxVel>
     <fdir1>1 0 0</fdir1>
   </gazebo>
-  <gazebo reference = "front_right_wheel_link">
+  <gazebo reference = "front_right_steering_link">
     <mu1>10000000</mu1>
     <mu2>10000000</mu2>
@@ -28,32 +55,5 @@
     <maxVel>10</maxVel>
     <fdir1>1 0 0</fdir1>
-  </gazebo>
-  <gazebo reference = "front_left_wheel_link">
-    <mu1>10000000</mu1>
-    <mu2>10000000</mu2>
-    <kp>10000000</kp>
-    <kd>10000000</kd>
-    <minDepth>0.001</minDepth>
-    <maxVel>10</maxVel>
-    <fdir1>1 0 0</fdir1>
-  </gazebo>
-  <gazebo reference = "front_left_steering_link">
-    <mu1>1</mu1>
-    <mu2>1</mu2>
-    <kp>10000000</kp>
-    <kd>10000000</kd>
-    <minDepth>0.001</minDepth>
-    <maxVel>10</maxVel>
-    <fdir1>1 0 0</fdir1>
-  </gazebo>
-  <gazebo reference = "front_right_steering_link">
-    <mu1>1</mu1>
-    <mu2>1</mu2>
-    <kp>10000000</kp>
-    <kd>10000000</kd>
-    <minDepth>0.001</minDepth>
-    <maxVel>10</maxVel>
-    <fdir1>1 0 0</fdir1>
-  </gazebo>
+  </gazebo> -->
   <gazebo>
     <plugin filename ="gz_ros2_control-system" name = "gz_ros2_control::GazeboSimROS2ControlPlugin">

File: src/robot_description/urdf/materials.xacro (robot description, xacro)
@@ -17,5 +17,5 @@
   </material>
   <material name="grey">
-    <color rgba="0 0 0 0.5" />
+    <color rgba="0.25 0.25 0.25 1.0" />
   </material>
 </robot>

File: src/robot_description/urdf/robot_core.xacro (robot description, xacro)
@@ -10,60 +10,94 @@
   <joint name="base_joint" type="fixed">
     <parent link="base_footprint" />
-    <child link="base_link" />
+    <child link="bottom_link" />
     <origin xyz="0 0 0" rpy="0 0 0" />
   </joint>
-  <!-- Base link of the robot -->
-  <link name="base_link">
-    <visual>
-      <origin xyz="0 0 0" rpy="0 0 0"/>
-      <geometry>
-        <box size="${box_length} ${box_width} ${box_height}" />
-      </geometry>
-      <material name="red"/>
-    </visual>
-    <collision>
-      <geometry>
-        <box size="${box_length} ${box_width} ${box_height}" />
-      </geometry>
-    </collision>
-    <xacro:inertial_box mass="${box_mass}" x="${box_length}" y="${box_width}" z="${box_height}">
+  <!-- Bottom link of the robot -->
+  <link name="bottom_link">
+    <visual>
+      <origin xyz="0 0 0" rpy="0 0 0"/>
+      <geometry>
+        <box size="${bottom_link_length} ${bottom_link_width} ${bottom_link_height}" />
+      </geometry>
+      <material name="grey"/>
+    </visual>
+    <collision>
+      <geometry>
+        <box size="${bottom_link_length} ${bottom_link_width} ${bottom_link_height}" />
+      </geometry>
+    </collision>
+    <xacro:inertial_box mass="${bottom_link_mass}" x="${bottom_link_length}" y="${bottom_link_width}" z="${bottom_link_height}">
       <origin xyz="0 0 0" rpy="0 0 0"/>
     </xacro:inertial_box>
   </link>
-  <!-- Rear Left Wheel link -->
-  <link name="rear_left_wheel_link">
-    <visual>
-      <origin xyz="0 0 0" rpy="0 0 0"/>
-      <geometry>
-        <cylinder radius="${wheel_radius}" length="${wheel_length}" />
-      </geometry>
-      <material name="black"/>
-    </visual>
-    <collision>
-      <origin xyz="0 0 0" rpy="0 0 0"/>
-      <geometry>
-        <cylinder radius="${wheel_radius}" length="${wheel_length}" />
-      </geometry>
-    </collision>
-    <xacro:inertial_cylinder mass="${wheel_mass}" length="${wheel_length}" radius="${wheel_radius}">
-      <origin xyz="0 0 0" rpy="0 0 0"/>
-    </xacro:inertial_cylinder>
-  </link>
-  <!-- Rear right wheel link -->
-  <link name="rear_right_wheel_link">
-    <visual>
-      <origin xyz="0 0 0" rpy="0 0 0"/>
-      <geometry>
-        <cylinder radius="${wheel_radius}" length="${wheel_length}" />
-      </geometry>
-      <material name="black"/>
-    </visual>
-    <collision>
-      <origin xyz="0 0 0" rpy="0 0 0"/>
-      <geometry>
-        <cylinder radius="${wheel_radius}" length="${wheel_length}" />
-      </geometry>
-    </collision>
-    <xacro:inertial_cylinder mass="${wheel_mass}" length="${wheel_length}" radius="${wheel_radius}">
+  <link name="front_left_wheel_connector">
+    <visual>
+      <origin xyz="0 0 0" rpy="0 0 0" />
+      <geometry>
+        <cylinder radius="${wheel_connector_radius}" length="${wheel_connector_length}" />
+      </geometry>
+      <material name="red"/>
+    </visual>
+    <collision>
+      <origin xyz="0 0 0" rpy="0 0 0" />
+      <geometry>
+        <cylinder radius="${wheel_connector_radius}" length="${wheel_connector_length}" />
+      </geometry>
+    </collision>
+    <xacro:inertial_cylinder mass="${wheel_connector_mass}" length="${wheel_connector_length}" radius="${wheel_connector_radius}">
+      <origin xyz="0 0 0" rpy="0 0 0"/>
+    </xacro:inertial_cylinder>
+  </link>
+  <link name="front_right_wheel_connector">
+    <visual>
+      <origin xyz="0 0 0" rpy="0 0 0" />
+      <geometry>
+        <cylinder radius="${wheel_connector_radius}" length="${wheel_connector_length}" />
+      </geometry>
+      <material name="red"/>
+    </visual>
+    <collision>
+      <origin xyz="0 0 0" rpy="0 0 0" />
+      <geometry>
+        <cylinder radius="${wheel_connector_radius}" length="${wheel_connector_length}" />
+      </geometry>
+    </collision>
+    <xacro:inertial_cylinder mass="${wheel_connector_mass}" length="${wheel_connector_length}" radius="${wheel_connector_radius}">
+      <origin xyz="0 0 0" rpy="0 0 0"/>
+    </xacro:inertial_cylinder>
+  </link>
+  <link name="rear_left_wheel_connector">
+    <visual>
+      <origin xyz="0 0 0" rpy="0 0 0" />
+      <geometry>
+        <cylinder radius="${wheel_connector_radius}" length="${wheel_connector_length}" />
+      </geometry>
+      <material name="red"/>
+    </visual>
+    <collision>
+      <origin xyz="0 0 0" rpy="0 0 0" />
+      <geometry>
+        <cylinder radius="${wheel_connector_radius}" length="${wheel_connector_length}" />
+      </geometry>
+    </collision>
+    <xacro:inertial_cylinder mass="${wheel_connector_mass}" length="${wheel_connector_length}" radius="${wheel_connector_radius}">
+      <origin xyz="0 0 0" rpy="0 0 0"/>
+    </xacro:inertial_cylinder>
+  </link>
+  <link name="rear_right_wheel_connector">
+    <visual>
+      <origin xyz="0 0 0" rpy="0 0 0" />
+      <geometry>
+        <cylinder radius="${wheel_connector_radius}" length="${wheel_connector_length}" />
+      </geometry>
+      <material name="red"/>
+    </visual>
+    <collision>
+      <origin xyz="0 0 0" rpy="0 0 0" />
+      <geometry>
+        <cylinder radius="${wheel_connector_radius}" length="${wheel_connector_length}" />
+      </geometry>
+    </collision>
+    <xacro:inertial_cylinder mass="${wheel_connector_mass}" length="${wheel_connector_length}" radius="${wheel_connector_radius}">
       <origin xyz="0 0 0" rpy="0 0 0"/>
     </xacro:inertial_cylinder>
@@ -102,9 +136,7 @@
       </geometry>
     </collision>
-    <inertial>
-      <mass value="0.01" />
-      <origin xyz="0 0 0" />
-      <inertia ixx="0.0" ixy="0.0" ixz="0.0" iyy="0.0" iyz="0.0" izz="0.0" />
-    </inertial>
+    <xacro:inertial_cylinder mass="0.001" length="0.001" radius="0.01">
+      <origin xyz="0 0 0" rpy="0 0 0"/>
+    </xacro:inertial_cylinder>
   </link>
   <!-- Front right wheel -->
@@ -141,27 +173,56 @@
       </geometry>
     </collision>
-    <inertial>
-      <mass value="0.01" />
-      <origin xyz="0 0 0" />
-      <inertia ixx="0.0" ixy="0.0" ixz="0.0" iyy="0.0" iyz="0.0" izz="0.0" />
-    </inertial>
-  </link>
-  <!-- Joints-->
-  <joint name="rear_left_wheel_joint" type="continuous">
-    <parent link="base_link" />
-    <child link="rear_left_wheel_link" />
-    <origin xyz="-${box_length/2} ${(box_width/2)+(wheel_length/2)} -${box_height/2}" rpy="-${3.14159/2} 0 0" />
-    <axis xyz="0 0 1" />
-  </joint>
-  <joint name="rear_right_wheel_joint" type="continuous">
-    <parent link="base_link" />
-    <child link="rear_right_wheel_link" />
-    <origin xyz="-${box_length/2} -${(box_width/2)+(wheel_length/2)} -${box_height/2}" rpy="-${3.14159/2} 0 0" />
-    <axis xyz="0 0 1" />
+    <xacro:inertial_cylinder mass="0.001" length="0.001" radius="0.01">
+      <origin xyz="0 0 0" rpy="0 0 0"/>
+    </xacro:inertial_cylinder>
+  </link>
+  <!-- Rear Left Wheel-->
+  <link name="rear_left_wheel_link">
+    <visual>
+      <origin xyz="0 0 0" rpy="0 0 0"/>
+      <geometry>
+        <cylinder radius="${wheel_radius}" length="${wheel_length}" />
+      </geometry>
+      <material name="black"/>
+    </visual>
+    <collision>
+      <origin xyz="0 0 0" rpy="0 0 0"/>
+      <geometry>
+        <cylinder radius="${wheel_radius}" length="${wheel_length}" />
+      </geometry>
+    </collision>
+    <xacro:inertial_cylinder mass="${wheel_mass}" length="${wheel_length}" radius="${wheel_radius}">
+      <origin xyz="0 0 0" rpy="0 0 0"/>
+    </xacro:inertial_cylinder>
+  </link>
+  <!-- Rear right wheel -->
+  <link name="rear_right_wheel_link">
+    <visual>
+      <origin xyz="0 0 0" rpy="0 0 0"/>
+      <geometry>
+        <cylinder radius="${wheel_radius}" length="${wheel_length}" />
+      </geometry>
+      <material name="black"/>
+    </visual>
+    <collision>
+      <origin xyz="0 0 0" rpy="0 0 0"/>
+      <geometry>
+        <cylinder radius="${wheel_radius}" length="${wheel_length}" />
+      </geometry>
+    </collision>
+    <xacro:inertial_cylinder mass="${wheel_mass}" length="${wheel_length}" radius="${wheel_radius}">
+      <origin xyz="0 0 0" rpy="0 0 0"/>
+    </xacro:inertial_cylinder>
+  </link>
+  <!-- Bottom Joints-->
+  <joint name="front_left_wheel_connector_joint" type="fixed">
+    <parent link="bottom_link" />
+    <child link="front_left_wheel_connector" />
+    <origin xyz="${bottom_link_length/2-0.05} ${bottom_link_width/2} 0" rpy="-${3.1459/2} 0 0" />
   </joint>
   <joint name="front_left_steering_joint" type="revolute">
-    <parent link="base_link" />
+    <parent link="front_left_wheel_connector" />
     <child link="front_left_steering_link" />
-    <origin xyz="${box_length/2} ${(box_width/2)+(wheel_length/2)} -${box_height/2}" rpy="-${3.14159/2} 0 0" />
+    <origin xyz="0 0 ${wheel_connector_length/2}" rpy="0 0 0" />
     <axis xyz="0 1 0" />
     <limit lower="-1.0" upper="1.0" effort="100" velocity="100" />
@@ -172,10 +233,15 @@
     <origin xyz="0 0 0" rpy="0 0 0" />
     <axis xyz="0 0 1" />
-    <limit lower="-1.0" upper="1.0" effort="100" velocity="100" />
+    <limit effort="100" velocity="100" />
+  </joint>
+  <joint name="front_right_wheel_connector_joint" type="fixed">
+    <parent link="bottom_link" />
+    <child link="front_right_wheel_connector" />
+    <origin xyz="${bottom_link_length/2-0.05} -${bottom_link_width/2} 0" rpy="-${3.1459/2} 0 0" />
   </joint>
   <joint name="front_right_steering_joint" type="revolute">
-    <parent link="base_link" />
+    <parent link="front_right_wheel_connector" />
     <child link="front_right_steering_link" />
-    <origin xyz="${box_length/2} -${(box_width/2)+(wheel_length/2)} -${(box_height/2)}" rpy="-${3.14159/2} 0 0" />
+    <origin xyz="0 0 -${wheel_connector_length/2}" rpy="0 0 0" />
     <axis xyz="0 1 0" />
     <limit lower="-1.0" upper="1.0" effort="100" velocity="100" />
@@ -186,5 +252,152 @@
     <origin xyz="0 0 0" rpy="0 0 0" />
     <axis xyz="0 0 1" />
-    <limit lower="-1.0" upper="1.0" effort="100" velocity="100" />
-  </joint>
+    <limit effort="100" velocity="100" />
+  </joint>
+  <joint name="rear_left_wheel_connector_joint" type="fixed">
+    <parent link="bottom_link" />
+    <child link="rear_left_wheel_connector" />
+    <origin xyz="-${bottom_link_length/2-0.05} ${bottom_link_width/2} 0" rpy="-${3.1459/2} 0 0" />
+  </joint>
+  <joint name="rear_right_wheel_connector_joint" type="fixed">
+    <parent link="bottom_link" />
+    <child link="rear_right_wheel_connector" />
+    <origin xyz="-${bottom_link_length/2-0.05} -${bottom_link_width/2} 0" rpy="-${3.1459/2} 0 0" />
+  </joint>
+  <joint name="rear_left_wheel_joint" type="continuous">
+    <parent link="rear_left_wheel_connector" />
+    <child link="rear_left_wheel_link" />
+    <origin xyz="0 0 ${wheel_connector_length/2}" rpy="0 0 0" />
+    <axis xyz="0 0 1" />
+    <limit effort="100" velocity="100" />
+  </joint>
+  <joint name="rear_right_wheel_joint" type="continuous">
+    <parent link="rear_right_wheel_connector" />
+    <child link="rear_right_wheel_link" />
+    <origin xyz="0 0 -${wheel_connector_length/2}" rpy="0 0 0" />
+    <axis xyz="0 0 1" />
+    <limit effort="100" velocity="100" />
+  </joint>
+  <!-- -->
+  <!-- -->
+  <!-- TOP LINKS -->
+  <link name="top_link">
+    <visual>
+      <origin xyz="0 0 0" rpy="0 0 0"/>
+      <geometry>
+        <box size="${top_link_length} ${top_link_width} ${top_link_height}" />
+      </geometry>
+      <material name="grey"/>
+    </visual>
+    <collision>
+      <geometry>
+        <box size="${top_link_length} ${top_link_width} ${top_link_height}" />
+      </geometry>
+    </collision>
+    <xacro:inertial_box mass="${top_link_mass}" x="${top_link_length}" y="${top_link_width}" z="${top_link_height}">
+      <origin xyz="0 0 0" rpy="0 0 0"/>
+    </xacro:inertial_box>
+  </link>
+  <link name="front_left_to_top_connector">
+    <visual>
+      <origin xyz="0 0 ${bottom_to_top_connector_length/2}" rpy="0 0 0" />
+      <geometry>
+        <cylinder radius="${bottom_to_top_connector_radius}" length="${bottom_to_top_connector_length}" />
+      </geometry>
+      <material name="red"/>
+    </visual>
+    <collision>
+      <origin xyz="0 0 ${bottom_to_top_connector_length/2}" rpy="0 0 0" />
+      <geometry>
+        <cylinder radius="${bottom_to_top_connector_radius}" length="${bottom_to_top_connector_length}" />
+      </geometry>
+    </collision>
+    <xacro:inertial_cylinder mass="${bottom_to_top_connector_mass}" length="${bottom_to_top_connector_length}" radius="${bottom_to_top_connector_radius}">
+      <origin xyz="0 0 0" rpy="0 0 0"/>
+    </xacro:inertial_cylinder>
+  </link>
+  <link name="front_right_to_top_connector">
+    <visual>
+      <origin xyz="0 0 ${bottom_to_top_connector_length/2}" rpy="0 0 0" />
+      <geometry>
+        <cylinder radius="${bottom_to_top_connector_radius}" length="${bottom_to_top_connector_length}" />
+      </geometry>
+      <material name="red"/>
+    </visual>
+    <collision>
+      <origin xyz="0 0 ${bottom_to_top_connector_length/2}" rpy="0 0 0" />
+      <geometry>
+        <cylinder radius="${bottom_to_top_connector_radius}" length="${bottom_to_top_connector_length}" />
+      </geometry>
+    </collision>
+    <xacro:inertial_cylinder mass="${bottom_to_top_connector_mass}" length="${bottom_to_top_connector_length}" radius="${bottom_to_top_connector_radius}">
+      <origin xyz="0 0 0" rpy="0 0 0"/>
+    </xacro:inertial_cylinder>
+  </link>
+  <link name="rear_left_to_top_connector">
+    <visual>
+      <origin xyz="0 0 ${bottom_to_top_connector_length/2}" rpy="0 0 0" />
+      <geometry>
+        <cylinder radius="${bottom_to_top_connector_radius}" length="${bottom_to_top_connector_length}" />
+      </geometry>
+      <material name="red"/>
+    </visual>
+    <collision>
+      <origin xyz="0 0 ${bottom_to_top_connector_length/2}" rpy="0 0 0" />
+      <geometry>
+        <cylinder radius="${bottom_to_top_connector_radius}" length="${bottom_to_top_connector_length}" />
+      </geometry>
+    </collision>
+    <xacro:inertial_cylinder mass="${bottom_to_top_connector_mass}" length="${bottom_to_top_connector_length}" radius="${bottom_to_top_connector_radius}">
+      <origin xyz="0 0 0" rpy="0 0 0"/>
+    </xacro:inertial_cylinder>
+  </link>
+  <link name="rear_right_to_top_connector">
+    <visual>
+      <origin xyz="0 0 ${bottom_to_top_connector_length/2}" rpy="0 0 0" />
+      <geometry>
+        <cylinder radius="${bottom_to_top_connector_radius}" length="${bottom_to_top_connector_length}" />
+      </geometry>
+      <material name="red"/>
+    </visual>
+    <collision>
+      <origin xyz="0 0 ${bottom_to_top_connector_length/2}" rpy="0 0 0" />
+      <geometry>
+        <cylinder radius="${bottom_to_top_connector_radius}" length="${bottom_to_top_connector_length}" />
+      </geometry>
+    </collision>
+    <xacro:inertial_cylinder mass="${bottom_to_top_connector_mass}" length="${bottom_to_top_connector_length}" radius="${bottom_to_top_connector_radius}">
+      <origin xyz="0 0 0" rpy="0 0 0"/>
+    </xacro:inertial_cylinder>
+  </link>
+  <!--TOP JOINTS-->
+  <joint name="front_left_bottom_joint" type="fixed">
+    <parent link="bottom_link" />
+    <child link="front_left_to_top_connector" />
+    <origin xyz="${bottom_link_length/2-0.05} ${bottom_link_width/2-0.05} 0" rpy="0 0 0" />
+  </joint>
+  <joint name="front_right_bottom_joint" type="fixed">
+    <parent link="bottom_link" />
+    <child link="front_right_to_top_connector" />
+    <origin xyz="${bottom_link_length/2-0.05} -${bottom_link_width/2-0.05} 0" rpy="0 0 0" />
+  </joint>
+  <joint name="rear_left_bottom_joint" type="fixed">
+    <parent link="bottom_link" />
+    <child link="rear_left_to_top_connector" />
+    <origin xyz="-${bottom_link_length/2-0.05} ${bottom_link_width/2-0.05} 0" rpy="0 0 0" />
+  </joint>
+  <joint name="rear_right_bottom_joint" type="fixed">
+    <parent link="bottom_link" />
+    <child link="rear_right_to_top_connector" />
+    <origin xyz="-${bottom_link_length/2-0.05} -${bottom_link_width/2-0.05} 0" rpy="0 0 0" />
+  </joint>
+  <joint name="front_left_top_joint" type="fixed">
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
File: src/robot_description/urdf/robot_physical_properties.xacro (robot description, xacro)
@@ -1,10 +1,20 @@
 <?xml version="1.0"?>
 <robot xmlns:xacro="http://ros.org/wiki/xacro">
-  <xacro:property name="wheel_radius" value="0.03" />
+  <xacro:property name="wheel_radius" value="0.05" />
   <xacro:property name="wheel_length" value="0.03" />
   <xacro:property name="wheel_mass" value="0.2" />
-  <xacro:property name="box_length" value="0.5" />
-  <xacro:property name="box_width" value="0.3" />
-  <xacro:property name="box_height" value="0.1" />
-  <xacro:property name="box_mass" value="1.0" />
+  <xacro:property name="bottom_link_length" value="0.5" />
+  <xacro:property name="bottom_link_width" value="0.3" />
+  <xacro:property name="bottom_link_height" value="0.02" />
+  <xacro:property name="bottom_link_mass" value="1.0" />
+  <xacro:property name="top_link_length" value="0.5" />
+  <xacro:property name="top_link_width" value="0.3" />
+  <xacro:property name="top_link_height" value="0.02" />
+  <xacro:property name="top_link_mass" value="1.0" />
+  <xacro:property name="wheel_connector_length" value="0.1" />
+  <xacro:property name="wheel_connector_radius" value="0.01" />
+  <xacro:property name="wheel_connector_mass" value="0.01" />
+  <xacro:property name="bottom_to_top_connector_length" value="0.1" />
+  <xacro:property name="bottom_to_top_connector_radius" value="0.005" />
+  <xacro:property name="bottom_to_top_connector_mass" value="0.01"/>
 </robot>
